File: pcb/102/uradmonitor_D.brd (EAGLE design)
At the start: 109 x 61 mm, 103 parts, among them IC2 MEGA128-A, IC4 TP4056, IC5 BME280, Q2 SI2305, T1 MMBT2907, T2 MPSA42, T3 MMBT2222, T4 2907, T5 MMBT2907, T7 MMBT2222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

Commit message: 12pF caps to 16MHz crystal
Parts:
- C1, C2: value 22pF -> 12pF
